File: Charming/Charming.sch (KiCad schematic (older format))
At the start: 97 parts, among them SW1 SW_Push, SW10 SW_Push, SW11 SW_Push, SW12 SW_Push, SW13 SW_Push, SW14 SW_Push, SW15 SW_Push, SW16 SW_Push, SW17 SW_Push, SW18 SW_Push, SW19 SW_Push, SW2 SW_Push, SW20 SW_Push, SW21 SW_Push, SW22 SW_Push, SW23 SW_Push, SW24 SW_Push, SW25 SW_Push, SW26 SW_Push, SW27 SW_Push, SW28 SW_Push, SW29 SW_Push, SW3 SW_Push, SW30 SW_Push, SW31 SW_Push, SW32 SW_Push, SW33 SW_Push, SW34 SW_Push, SW35 SW_Push, SW36 SW_Push, SW37 SW_Push, SW38 SW_Push, SW39 SW_Push, SW4 SW_Push, SW40 SW_Push, SW41 SW_Push, SW42 SW_Push, SW43 SW_Push, SW44 SW_Push, SW45 SW_Push, SW46 SW_Push, SW47 SW_Push, SW48 SW_Push, SW5 SW_Push, SW6 SW_Push, SW7 SW_Push, SW8 SW_Push, SW9 SW_Push, U1 ProMicro

Commit message: v2
Changed lines of the file:
@@
 encoding utf-8
 Sheet 1 1
-Title "Charming"
-Date "2020-06-18"
-Rev "1.0"
+Title "Charming 40"
+Date "2020-06-21"
+Rev "2"
 Comp "Designed by James Sa"
 Comment1 ""
@@
 Text GLabel 2200 2350 0    50   Input ~ 0
 row3
-Text GLabel 3600 2350 2    50   Input ~ 0
+Text GLabel 3600 2150 2    50   Input ~ 0
 col6
-Text GLabel 3600 2250 2    50   Input ~ 0
+Text GLabel 3600 2050 2    50   Input ~ 0
 col7
-Text GLabel 3600 2050 2    50   Input ~ 0
+Text GLabel 3600 1950 2    50   Input ~ 0
 col8
-Text GLabel 3600 1950 2    50   Input ~ 0
+Text GLabel 3600 1850 2    50   Input ~ 0
 col9
-Text GLabel 3600 1850 2    50   Input ~ 0
+Text GLabel 3600 1750 2    50   Input ~ 0
 col10
-Text GLabel 3600 1750 2    50   Input ~ 0
+Text GLabel 3600 1650 2    50   Input ~ 0
 col11
 NoConn ~ 3600 1450
@@
 	1    0    0    -1
 $EndComp
+Text GLabel 3600 2250 2    50   Input ~ 0
+col5
+Text GLabel 3600 2350 2    50   Input ~ 0
+col4
 Text GLabel 2200 2150 0    50   Input ~ 0
-col5
+col3
 Text GLabel 2200 2050 0    50   Input ~ 0
-col4
+col2
+Text GLabel 2200 1850 0    50   Input ~ 0
+col0
+Text GLabel 2200 1750 0    50   Input ~ 0
+row1
 Text GLabel 2200 1950 0    50   Input ~ 0
-col3
-Text GLabel 2200 1850 0    50   Input ~ 0
-col2
+col1
+Wire Wire Line
+	3600 1350 4150 1350
 Text GLabel 2200 1650 0    50   Input ~ 0
-col0
-Text GLabel 3600 2150 2    50   Input ~ 0
-row1
-Text GLabel 2200 1750 0    50   Input ~ 0
-col1
-Wire Wire Line
-	3600 1350 4150 1350
-Text GLabel 3600 1650 2    50   Input ~ 0
 row0
 $Comp
