File: Charming/Charming.sch (KiCad schematic (older format))
At the start: 97 parts, among them SW1 SW_Push, SW10 SW_Push, SW11 SW_Push, SW12 SW_Push, SW13 SW_Push, SW14 SW_Push, SW15 SW_Push, SW16 SW_Push, SW17 SW_Push, SW18 SW_Push, SW19 SW_Push, SW2 SW_Push, SW20 SW_Push, SW21 SW_Push, SW22 SW_Push, SW23 SW_Push, SW24 SW_Push, SW25 SW_Push, SW26 SW_Push, SW27 SW_Push, SW28 SW_Push, SW29 SW_Push, SW3 SW_Push, SW30 SW_Push, SW31 SW_Push, SW32 SW_Push, SW33 SW_Push, SW34 SW_Push, SW35 SW_Push, SW36 SW_Push, SW37 SW_Push, SW38 SW_Push, SW39 SW_Push, SW4 SW_Push, SW40 SW_Push, SW41 SW_Push, SW42 SW_Push, SW43 SW_Push, SW44 SW_Push, SW45 SW_Push, SW46 SW_Push, SW47 SW_Push, SW48 SW_Push, SW5 SW_Push, SW6 SW_Push, SW7 SW_Push, SW8 SW_Push, SW9 SW_Push, U1 ProMicro

Commit message: even odd pins
Changed lines of the file:
@@
 Text GLabel 2200 2350 0    50   Input ~ 0
 row3
+Text GLabel 3600 1950 2    50   Input ~ 0
+col6
+Text GLabel 2200 2050 0    50   Input ~ 0
+col7
 Text GLabel 3600 2150 2    50   Input ~ 0
-col6
-Text GLabel 3600 2050 2    50   Input ~ 0
-col7
-Text GLabel 3600 1950 2    50   Input ~ 0
 col8
-Text GLabel 3600 1850 2    50   Input ~ 0
+Text GLabel 2200 2150 0    50   Input ~ 0
 col9
-Text GLabel 3600 1750 2    50   Input ~ 0
+Text GLabel 3600 2250 2    50   Input ~ 0
 col10
-Text GLabel 3600 1650 2    50   Input ~ 0
+Text GLabel 2200 2250 0    50   Input ~ 0
 col11
 NoConn ~ 3600 1450
@@
 	1    0    0    -1
 $EndComp
-Text GLabel 3600 2250 2    50   Input ~ 0
+Text GLabel 2200 1950 0    50   Input ~ 0
 col5
-Text GLabel 3600 2350 2    50   Input ~ 0
+Text GLabel 3600 1850 2    50   Input ~ 0
 col4
-Text GLabel 2200 2150 0    50   Input ~ 0
+Text GLabel 2200 1850 0    50   Input ~ 0
 col3
-Text GLabel 2200 2050 0    50   Input ~ 0
+Text GLabel 3600 1750 2    50   Input ~ 0
 col2
-Text GLabel 2200 1850 0    50   Input ~ 0
+Text GLabel 3600 1650 2    50   Input ~ 0
 col0
+Text GLabel 3600 2050 2    50   Input ~ 0
+row1
 Text GLabel 2200 1750 0    50   Input ~ 0
-row1
-Text GLabel 2200 1950 0    50   Input ~ 0
 col1
 Wire Wire Line
@@
 Wire Wire Line
 	4000 1550 3600 1550
-Text GLabel 2200 2250 0    50   Input ~ 0
+Text GLabel 3600 2350 2    50   Input ~ 0
 row2
 $EndSCHEMATC

Commit message: new layout
Parts:
- removed D1: D, Diode_SMD:D_SOD-123, symbol Diode:1N4148W
- removed D10, D11, D12, D13, D14, D15, D16, D17, D18, D19, D2, D20, D21, D22, D23, D24, D25, D26, D27, D28, D29, D3, D30, D31, D32, D33, D34, D35, D36, D37, D38, D39, D40, D41, D42, D43, D44, D45, D46, D47, D48, D8, D9: D, Diode_SMD:D_SOD-123, symbol Device:D
- removed SW10, SW11, SW12, SW13, SW14, SW15, SW16, SW17, SW18, SW19, SW20, SW21, SW22, SW23, SW24, SW25, SW26, SW27, SW28, SW29, SW30, SW31, SW32, SW33, SW34, SW35, SW36, SW37, SW38, SW39, SW40, SW41, SW42, SW43, SW44, SW45, SW46, SW47, SW48, SW5, SW6, SW7, SW8, SW9: SW_Push, Charming:SW_PG1350, symbol Switch:SW_Push
- removed U1: ProMicro, Keebio:ArduinoProMicro, symbol keebio:ProMicro
- added Boot1: Boot, Button_Switch_THT:SW_PUSH_6mm, symbol Switch:SW_Push
- added C1: 4.7u, Capacitor_THT:CP_Radial_D4.0mm_P1.50mm, symbol Device:CP
- added C2, C3: 0.1u, Capacitor_THT:C_Disc_D4.3mm_W1.9mm_P5.00mm, symbol Device:C
- added C4, C5: 22pf, Capacitor_THT:C_Disc_D3.0mm_W1.6mm_P2.50mm, symbol Device:C
- added D1: LED, LED_THT:LED_D3.0mm, symbol Device:LED
- added D2, D3: 3.6V, Diode_THT:D_DO-35_SOD27_P7.62mm_Horizontal, symbol Device:D_Zener
- added F1: 100mA, Fuse:Fuse_Bourns_MF-RG500, symbol Device:Polyfuse
- added J1: AVR-ISP-6, Keebio:ICSP-Header, symbol Connector:AVR-ISP-6
- added R1: 10k, Resistor_THT:R_Axial_DIN0204_L3.6mm_D1.6mm_P5.08mm_Horizontal, symbol Device:R
- added R2: 1.5K, Resistor_THT:R_Axial_DIN0204_L3.6mm_D1.6mm_P5.08mm_Horizontal, symbol Device:R
- added R3, R4: 5.1K, Resistor_THT:R_Axial_DIN0204_L3.6mm_D1.6mm_P5.08mm_Horizontal, symbol Device:R
- added R5, R6: 75, Resistor_THT:R_Axial_DIN0204_L3.6mm_D1.6mm_P5.08mm_Horizontal, symbol Device:R
- added Reset1: Reset, Button_Switch_THT:SW_PUSH_6mm, symbol Switch:SW_Push
- added U1: ATmega328P-PU, Package_DIP:DIP-28_W7.62mm, symbol MCU_Microchip_ATmega:ATmega328P-PU
- added USB1: HRO-TYPE-C-31-M-12, Keebio:HRO-TYPE-C-31-M-12-Assembly, symbol Charming-rescue:HRO-TYPE-C-31-M-12-keebio
- added Y1: 16MHz, Crystal:Crystal_HC49-4H_Vertical, symbol Device:Crystal
- D4, D5, D6, D7: footprint Diode_SMD:D_SOD-123 -> Diode_THT:D_DO-35_SOD27_P7.62mm_Horizontal
- SW1, SW2, SW3, SW4: footprint Charming:SW_PG1350 -> Button_Switch_Keyboard:SW_Cherry_MX_1.00u_PCB
Connections:
- net labels added: +5V, Boot, Col0, Col1, D+, D-, Miso, Mosi, Reset, Row0, Row1, Sck
- net labels removed: VCC, col0, col1, col10, col11, col2, col3, col4, col5, col6, col7, col8, col9, row0, row1, row2, row3
- wire segments 113 -> 65
- no-connect marks 4 -> 13

Commit message: customize symbol and footprint
Parts:
- J1: value AVR-ISP-6 -> AVR ISP; footprint Keebio:ICSP-Header -> Charming:AVRISP; symbol Connector:AVR-ISP-6 -> Charming:Oshwa_ISP_6
- USB1: value HRO-TYPE-C-31-M-12 -> TYPE-C; footprint Keebio:HRO-TYPE-C-31-M-12-Assembly -> Charming:USB_C_Receptacle_HRO_TYPE-C-31-M-12; symbol Charming-rescue:HRO-TYPE-C-31-M-12-keebio -> Charming:USB-2.0-Type-C-Receptacle
Connections:
- net GND: now also R4.2, USB1.A1 (GND), USB1.B1 (GND), USB1.S1 (SHIELD); no longer R4.1, USB1.1 (GND), USB1.12 (GND), USB1.13 (SHIELD)
- net at R3.2: now also USB1.A5 (CC1); no longer USB1.4 (CC1)
- net at D3.1 (K), R6.1: now also USB1.A7 (D-), USB1.B7 (D-); no longer USB1.5 (DN2), USB1.7 (DN1)
- net at D2.1 (K), R5.2: now also USB1.A6 (D+), USB1.B6 (D+); no longer USB1.6 (DP1), USB1.8 (DP2)
- net Miso renamed SDO
- net Mosi renamed SDI
- net Sck renamed SCK
- new net: F1.2, USB1.A4 (VBUS), USB1.B4 (VBUS)
- new net: R4.1, USB1.B5 (CC2)
Other:
- note added: "SDO – Serial Data Out. An output signal on a device where data is sent out to another SPI device. Replace MOSI\nSDI – Serial Data In. An input signal on a device where data is received from another SPI device. Replace MISO\nCS – Chip Select. Activated by the controller to initiate communication with a given peripheral. Replace SS\n\nDetails here: https://www.oshwa.org/a-resolution-to-redefine-spi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"
- moved on the sheet: D2, D3, J1, R3, R4, R5, R6

Commit message: name netlist
Connections:
- net VSUB: now reaches F1.2, USB1.A4 (VBUS), USB1.B4 (VBUS)
- net CC1: now reaches R3.2, USB1.A5 (CC1)
- net DP: now reaches D2.1 (K), R5.2, USB1.A6 (D+), USB1.B6 (D+)
- net DN: now reaches D3.1 (K), R6.1, USB1.A7 (D-), USB1.B7 (D-)
- net CC2: now reaches R4.1, USB1.B5 (CC2)
Changed lines of the file:
@@
 Wire Wire Line
 	6300 4100 6300 4200
+Text Label 6200 3200 0    50   ~ 0
+DP
+Text Label 6200 3400 0    50   ~ 0
+DN
+Text Label 6000 2850 0    50   ~ 0
+VSUB
+Text Label 5700 3600 0    50   ~ 0
+CC1
+Text Label 5700 3700 0    50   ~ 0
+CC2
 $EndSCHEMATC

Commit message: move customize footprints to external libs
Parts:
- J1: footprint Charming:AVRISP -> JSA:AVRISP; symbol Charming:Oshwa_ISP_6 -> JSA:Oshwa_ISP_6
- USB1: footprint Charming:USB_C_Receptacle_HRO_TYPE-C-31-M-12 -> JSA:USB_C_Receptacle_HRO_TYPE-C-31-M-12; symbol Charming:USB-2.0-Type-C-Receptacle -> JSA:USB-2.0-Type-C-Receptacle
Changed lines of the file:
@@
 Reset
 $Comp
-L Charming:Oshwa_ISP_6 J1
+L JSA:Oshwa_ISP_6 J1
 U 1 1 5F1679A9
 P 4000 5200
 F 0 "J1" H 3671 5296 50  0000 R CNN
 F 1 "AVR ISP" H 3671 5205 50  0000 R CNN
-F 2 "Charming:AVRISP" V 3750 5250 50  0001 C CNN
-F 3 " ~" H 2725 4650 50  0001 C CNN
+F 2 "JSA:AVRISP" V 3750 5250 50  0001 C CNN
+F 3 "https://www.oshwa.org/a-resolution-to-redefine-spi-signal-names" H 2725 4650 50  0001 C CNN
 	1    4000 5200
 	1    0    0    -1
@@
 	5700 4000 5800 4000
 $Comp
-L Charming:USB-2.0-Type-C-Receptacle USB1
+L JSA:USB-2.0-Type-C-Receptacle USB1
 U 1 1 5F11DCBC
 P 5600 3550
 F 0 "USB1" H 5372 3603 60  0000 R CNN
 F 1 "TYPE-C" H 5372 3497 60  0000 R TNN
-F 2 "Charming:USB_C_Receptacle_HRO_TYPE-C-31-M-12" H 5600 3550 60  0001 C CNN
+F 2 "JSA:USB_C_Receptacle_HRO_TYPE-C-31-M-12" H 5600 3550 60  0001 C CNN
 F 3 "" H 5600 3550 60  0001 C CNN
 	1    5600 3550
