File: Charming/Charming.kicad_pcb (KiCad board)
At the start: 2 copper layers, 29 parts, among them J1 AVR ISP, SW1 SW_Push, SW2 SW_Push, SW3 SW_Push, SW4 SW_Push, U1 ATmega328P-PU, Y1 16MHz

Commit message: power first design
Parts:
- moved F1 16.3 mm to (46.1, 85.9), turned to 270 degrees
- moved D1 13.9 mm to (50.7, 85.7), turned to 0 degrees
- moved D3 13.6 mm to (52.0, 99.8)
- moved R6 12.1 mm to (58.4, 99.6)
- moved R2 10.1 mm to (63.5, 87.7)
- moved C1 8.57 mm to (51.9, 90.7), turned to 270 degrees
- moved R1 8.15 mm to (58.7, 90.1), turned to 0 degrees
- moved D2 6.50 mm to (52.5, 96.3)
- moved R5 6.41 mm to (63.5, 96.4)
- moved C4 1.86 mm to (103.0, 97.9)
- moved R3 1.59 mm to (63.5, 85.4)
- moved R4 1.11 mm to (58.7, 92.5)
- moved Reset1 0.92 mm to (115.0, 84.5)
Routing:
- net Net-(D6-Pad2): track 97.4 -> 0.00 mm
- net Net-(D4-Pad2): track 90.4 -> 0.00 mm
- net Net-(D7-Pad2): track 82.3 -> 0.00 mm
- net Col1: track 73.1 -> 0.00 mm
- net Net-(D5-Pad2): track 72.3 -> 0.00 mm
- net SCK: track 66.3 -> 0.00 mm
- net +5V: track 0.00 -> 64.3 mm
- net SDI: track 63.0 -> 0.00 mm
- net SDO: track 62.2 -> 0.00 mm
- net Col0: track 52.8 -> 0.00 mm
- net Reset: track 105.0 -> 56.1 mm
- net Row1: track 45.6 -> 0.00 mm
- net Row0: track 36.2 -> 0.00 mm
- net Net-(D3-Pad1): track 24.3 -> 35.3 mm
- net Net-(C4-Pad2): track 10.3 -> 0.00 mm
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
Commit message: name netlist
Parts:
- moved R2 4.68 mm to (58.8, 87.7), turned to 0 degrees
Connections:
- net Net-(D2-Pad1) renamed /DP
- net Net-(D3-Pad1) renamed /DN
- net Net-(F1-Pad2) renamed /VSUB
- net Net-(R3-Pad2) renamed /CC1
- net Net-(R4-Pad1) renamed /CC2
Routing:
- net +5V: track 64.3 -> 92.0 mm
- net Net-(D1-Pad2): track 5.76 -> 11.5 mm
- net /DP: track 33.2 -> 35.4 mm

Commit message: move customize footprints to external libs
Parts:
- J1: footprint Charming:AVRISP -> JSA:AVRISP
- USB1: footprint Charming:USB_C_Receptacle_HRO_TYPE-C-31-M-12 -> JSA:USB_C_Receptacle_HRO_TYPE-C-31-M-12
